File: LoRaShield2.sch (KiCad schematic (older format))
At the start: 24 parts, among them J1 SMA_EDGE, J2 Conn_02x20_Odd_Even, J3 Conn_02x06_Odd_Even, U1 RFM95PW, U2 TXB0108-DFN20, U3 TXB0108-DFN20

Commit message: update to rev2.1
Parts:
- removed NT1: Net-Tie_2, Oddities:NetTie-I_Connected_SMD, symbol Device:Net-Tie_2
- added C11: 1u, Capacitors_SMD:C_0603, symbol Device:C_Small
- added FID1, FID2, FID3: Fiducial, Fiducials:Fiducial_0.5mm_Dia_1mm_Outer, symbol Mechanical:Fiducial
- added J4: Conn_01x04, Pin_Headers:Pin_Header_Straight_1x04_Pitch2.54mm, symbol conn:Conn_01x04
- added R5: 0, Resistors_SMD:R_0402, symbol Device:R
- A1: footprint mogar_modules_new:Arduino_UNO_R3_WithMountingHoles -> mogar_modules_new:Arduino_UNO_HamShieldFootprint
Connections:
- net labels added: GPS_RX, GPS_TX
- wire segments 166 -> 178
Other:
- note added: "UBlox Neo 6M GPS Module Connections"
- moved on the sheet: A1, J3
